File: hardware/Longan Nano SIL Adapter.sch (EAGLE design)
At the start: 18 parts

Commit message: final schematics and routing
Parts:
- removed LF-COM-2: BEAD 500mA, 2021-07-02 OrangeHat Library:L-M2012
- added CB-COM-1: 1u, Passives:C-M2012
- CF-COM-1: value 100n 50v -> 100n; device 2021-07-02 OrangeHat Library:C-NPOL -> Passives:C-M2012
- CF-COM-2: value 100n 50V -> 100n; device 2021-07-02 OrangeHat Library:C-NPOL -> Passives:C-M2012
- CON-COM-1, CON-COM-2: device 2021-07-02 OrangeHat Library:JACK_SMD_3MM5 -> Library:JACK_SMD_3MM5
- LF1-COM-1: device 2021-07-02 OrangeHat Library:L-M2012 -> Passives:L-M2012
- RS-COM-2, RS-COM-3: device 2021-07-02 OrangeHat Library:R-M2012 -> Passives:R-M2012
- RS-UC-1: value RX4-M2012-X4 -> 4X1K
Connections:
- removed net V-485: CF-COM-2.1, IC-COM-1.V-, LF-COM-2.2, RD-COM-1.1, RS-COM-2.1, RS-COM-3.1
- net V+485: now also CB-COM-1.2
- net V-: now also CB-COM-1.1, CF-COM-2.1, IC-COM-1.V-, RD-COM-1.1, RS-COM-2.1, RS-COM-3.1; no longer LF-COM-2.1
